Commit message: Optimize reachability

File: data/robot_with_visuals.urdf (robot description, URDF)
Before this commit: robot robot_arm, 8 links, 7 joints
Links:
- link link5: geometry visual cylinder length=0.1 radius=0.05; visual cylinder length=0.2 radius=0.05
Joints:
- joint joint6: origin xyz=0 0.346 0 rpy=-1.570796 0 0 -> xyz=0 0.2 0 rpy=-1.570796 0 0
